Commit message: Fixed robot falling over immediately after starting up
fixed table & obstruction being pitch black

File: src/franka_sorting/description/franka_camera.urdf.xacro (robot description, xacro)
@@ -41,5 +41,55 @@
   </gazebo>
   <link name="world"/>
-  <xacro:panda_arm base_parent="world"/>
-  <xacro:panda_gripper wrist_flange="panda_link8"/>
+    <xacro:panda_arm base_parent="world"/>
+    <xacro:panda_gripper wrist_flange="panda_link8"/>
+    <ros2_control name="GazeboSimSystem" type="system">
+      <hardware>
+        <plugin>gz_ros2_control/GazeboSimSystem</plugin>
+      </hardware>
+      <joint name="panda_joint1">
+        <command_interface name="position"/>
+        <state_interface name="position"/>
+        <state_interface name="velocity"/>
+      </joint>
+      <joint name="panda_joint2">
+        <command_interface name="position"/>
+        <state_interface name="position"/>
+        <state_interface name="velocity"/>
+      </joint>
+      <joint name="panda_joint3">
+        <command_interface name="position"/>
+        <state_interface name="position"/>
+        <state_interface name="velocity"/>
+      </joint>
+      <joint name="panda_joint4">
+        <command_interface name="position"/>
+        <state_interface name="position"/>
+        <state_interface name="velocity"/>
+      </joint>
+      <joint name="panda_joint5">
+        <command_interface name="position"/>
+        <state_interface name="position"/>
+        <state_interface name="velocity"/>
+      </joint>
+      <joint name="panda_joint6">
+        <command_interface name="position"/>
+        <state_interface name="position"/>
+        <state_interface name="velocity"/>
+      </joint>
+      <joint name="panda_joint7">
+        <command_interface name="position"/>
+        <state_interface name="position"/>
+        <state_interface name="velocity"/>
+      </joint>
+    </ros2_control>
+  <gazebo>
+    <plugin filename="libgz_ros2_control-system.so" name="gz_ros2_control::GazeboSimROS2ControlPlugin">
+      <parameters>$(find franka_sorting)/config/franka_controllers.yaml</parameters>
+    </plugin>
+  </gazebo>
+  <gazebo>
+    <plugin filename="libgz_ros2_control-system.so" name="gz_ros2_control::GazeboSimROS2ControlPlugin">
+      <parameters>$(find franka_sorting)/config/franka_controllers.yaml</parameters>
+    </plugin>
+  </gazebo>
 </robot>

Commit message: finalizing setup for robot arm
able to command arm position & gripper open/close from command line using ros2 publishers now!

File: src/franka_sorting/description/franka_camera.urdf.xacro (robot description, xacro)
@@ -82,4 +82,14 @@
         <state_interface name="velocity"/>
       </joint>
+      <joint name="panda_finger_joint1">
+        <command_interface name="position"/>
+        <state_interface name="position"/>
+        <state_interface name="velocity"/>
+      </joint>
+      <joint name="panda_finger_joint2">
+        <command_interface name="position"/>
+        <state_interface name="position"/>
+        <state_interface name="velocity"/>
+      </joint>
     </ros2_control>
   <gazebo>
@@ -88,8 +98,3 @@
     </plugin>
   </gazebo>
-  <gazebo>
-    <plugin filename="libgz_ros2_control-system.so" name="gz_ros2_control::GazeboSimROS2ControlPlugin">
-      <parameters>$(find franka_sorting)/config/franka_controllers.yaml</parameters>
-    </plugin>
-  </gazebo>
 </robot>
