Commit message: Able to see image & depth_image out of RBGD camera now!

File: src/franka_sorting/description/franka.urdf.xacro (robot description, xacro)
@@ -1,44 +1,7 @@
 <?xml version="1.0"?>
 <robot xmlns:xacro="http://www.ros.org/wiki/xacro" name="franka_sorting_setup">
+  <link name="world"/>
   <xacro:include filename="$(find panda_description)/urdf/panda_arm.xacro"/>
   <xacro:include filename="$(find panda_description)/urdf/panda_gripper.xacro"/>
-  <link name="camera_link">
-    <visual>
-      <origin xyz="0 0 0" rpy="0 0 0"/>
-      <geometry>
-        <box size="0.05 0.05 0.03"/>
-      </geometry>
-      <material name="black">
-        <color rgba="0.1 0.1 0.1 1.0"/>
-      </material>
-    </visual>
-  </link>
-  <joint name="world_to_camera" type="fixed">
-    <parent link="world"/>
-    <child link="camera_link"/>
-    <origin xyz="0.6 0.0 1.2" rpy="0 1.5708 0"/>
-  </joint>
-  <gazebo reference="camera_link">
-    <sensor name="rgbd_camera" type="rgbd_camera">
-      <camera>
-        <horizontal_fov>1.047</horizontal_fov>
-        <image>
-          <width>640</width>
-          <height>480</height>
-          <format>R8G8B8</format>
-        </image>
-        <clip>
-          <near>0.1</near>
-          <far>10</far>
-        </clip>
-      </camera>
-      <always_on>1</always_on>
-      <update_rate>30</update_rate>
-      <visualize>true</visualize>
-      <topic>camera</topic>
-      <gz_frame_id>camera_link</gz_frame_id>
-    </sensor>
-  </gazebo>
-  <link name="world"/>
     <xacro:panda_arm base_parent="world"/>
     <xacro:panda_gripper wrist_flange="panda_link8"/>
