Commit message: x, y, z from block_detector now reflects pose in Gazebo

File: src/franka_sorting/description/camera_only.urdf.xacro (robot description, xacro)
@@ -15,8 +15,14 @@
     </inertial>
   </link>
+  <link name="camera_link_optical"/>
   <joint name="world_to_camera" type="fixed">
     <parent link="world"/>
     <child link="camera_link"/>
     <origin xyz="0.6 0.0 1.2" rpy="0 1.5708 0"/>
+  </joint>
+  <joint name="camera_optical_joint" type="fixed">
+    <parent link="camera_link"/>
+    <child link="camera_link_optical"/>
+    <origin xyz="0 0 0" rpy="-1.5708 0 -1.5708"/>
   </joint>
   <gazebo reference="camera_link">

Commit message: super epic awesome work session

File: src/franka_sorting/description/camera_only.urdf.xacro (robot description, xacro)
@@ -19,5 +19,5 @@
     <parent link="world"/>
     <child link="camera_link"/>
-    <origin xyz="0.6 0.0 1.2" rpy="0 1.5708 0"/>
+    <origin xyz="0.6 0.0 5.0" rpy="0 1.5708 0"/>
   </joint>
   <joint name="camera_optical_joint" type="fixed">

Commit message: robot arm moves, detected poses are off

File: src/franka_sorting/description/camera_only.urdf.xacro (robot description, xacro)
@@ -1,5 +1,4 @@
 <?xml version="1.0"?>
 <robot xmlns:xacro="http://www.ros.org/wiki/xacro" name="external_camera">
-  <link name="world"/>
   <link name="camera_link">
     <visual>
@@ -16,9 +15,4 @@
   </link>
   <link name="camera_link_optical"/>
-  <joint name="world_to_camera" type="fixed">
-    <parent link="world"/>
-    <child link="camera_link"/>
-    <origin xyz="0.6 0.0 5.0" rpy="0 1.5708 0"/>
-  </joint>
   <joint name="camera_optical_joint" type="fixed">
     <parent link="camera_link"/>

Commit message: fixed perception issues, arm picked up block for the first timegit add src/franka_sorting/launch/franka_sim.launch.py git add src/franka_sorting/launch/franka_sim.launch.py git add src/franka_sorting/launch/franka_sim.launch.py

File: src/franka_sorting/description/camera_only.urdf.xacro (robot description, xacro)
@@ -18,5 +18,5 @@
     <parent link="camera_link"/>
     <child link="camera_link_optical"/>
-    <origin xyz="0 0 0" rpy="-1.5708 0 -1.5708"/>
+    <origin xyz="0 0 0" rpy="-1.5708 0 1.5708"/>
   </joint>
   <gazebo reference="camera_link">

Commit message: can semi-reliably pick up and sort red obj.
red detection reappears after back in container

File: src/franka_sorting/description/camera_only.urdf.xacro (robot description, xacro)
@@ -18,5 +18,5 @@
     <parent link="camera_link"/>
     <child link="camera_link_optical"/>
-    <origin xyz="0 0 0" rpy="-1.5708 0 1.5708"/>
+    <origin xyz="0 0 0" rpy="-1.5708 0 -1.5708"/>
   </joint>
   <gazebo reference="camera_link">

File: src/franka_sorting/description/franka.urdf.xacro (robot description, xacro)
@@ -10,5 +10,5 @@
     	<parent link="world"/>
     	<child link="camera_link"/>
-    	<origin xyz="0.8 0.0 2.0" rpy="0 1.5708 0"/>
+    	<origin xyz="0.8 0.0 2.0" rpy="3.14159 1.5708 0"/>
     </joint>
     <ros2_control name="GazeboSimSystem" type="system">
